File: galspanic.kicad_sch (KiCad schematic)
At the start: 19 parts, among them J1 x68000_expansion, U1 CY62167E, U2 CY62167E, U3 CY62167E, U4 CY62167E, U5 CY62167E, U6 ATF22V10C-10XU

Commit message: Small Update
Added LCSC Part numbers
Extended Ground Plane
Replaced throughole capacitor with SMD capacitor
Removed vias on footprint pads
Changed via dimensions to 0.6/0.3
Added stitching vias
Rotated solder jumper text
Changed solder mask to black
Parts:
- C7: value 220uF -> (none); footprint Capacitor_THT:CP_Radial_D6.3mm_P2.50mm -> (none); LCSC Part (none) -> C340768
- JP1: value SolderJumper_3_Bridged12 -> (none); footprint Jumper:SolderJumper-3_P1.3mm_Bridged12_RoundedPad1.0x1.5mm -> (none)
